Commit message: Documentando Xacro

File: install/firebot_arm_pkg/share/firebot_arm_pkg/urdf/montagem.control.xacro (robot description, xacro)
@@ -3,17 +3,27 @@
   <!-- Configurações ros2_control para 3 juntas -->
   <ros2_control name="montagem_control" type="system">
+    <!-- Definição do plugin que conecta o controle ros2_control ao simulador Gazebo -->
     <hardware>
       <plugin>gazebo_ros2_control/GazeboSystem</plugin>
     </hardware>
+    <!-- Definição da primeira junta: linkvertical1_to_base_link -->
     <joint name="linkvertical1_to_base_link">
+      <!-- Interface de estado usada para monitorar a posição da junta -->
       <state_interface name="position"/>
+      <!-- Interface de comando usada para controlar a posição da junta -->
       <command_interface name="position"/>
     </joint>
+    <!-- Definição da segunda junta: linkvertical2_to_linkvertical1 -->
     <joint name="linkvertical2_to_linkvertical1">
+      <!-- Interface de estado usada para monitorar a posição da junta -->
       <state_interface name="position"/>
+      <!-- Interface de comando usada para controlar a posição da junta -->
       <command_interface name="position"/>
     </joint>
+    <!-- Definição da terceira junta: linkhorizontal1_to_linkvertical2 -->
     <joint name="linkhorizontal1_to_linkvertical2">
+      <!-- Interface de estado usada para monitorar a posição da junta -->
       <state_interface name="position"/>
+      <!-- Interface de comando usada para controlar a posição da junta -->
       <command_interface name="position"/>
     </joint>

File: install/firebot_arm_pkg/share/firebot_arm_pkg/urdf/montagem.xacro (robot description, xacro)
@@ -1,160 +1,161 @@
 <?xml version="1.0" ?>
 <robot name="montagem" xmlns:xacro="http://www.ros.org/wiki/xacro">
-<xacro:include filename="$(find firebot_arm_pkg)/urdf/materials.xacro" />
-<xacro:include filename="$(find firebot_arm_pkg)/urdf/montagem.trans" />
-<xacro:include filename="$(find firebot_arm_pkg)/urdf/montagem.gazebo" />
-<xacro:include filename="$(find firebot_arm_pkg)/urdf/montagem.control.xacro" />
-<!-- Variáveis adicionadas -->
-<!-- <xacro:property name="base_to_vertical1_xyz" value="0.0 0.0 0.012"/>
-<xacro:property name="base_to_vertical1_rpy" value="0 0 0"/>
-<xacro:property name="vertical1_to_vertical2_xyz" value="0.105 0.105 0.71"/>
-<xacro:property name="vertical1_to_vertical2_rpy" value="0 0 0"/>
-<xacro:property name="vertical2_to_horizontal1_xyz" value="-0.17 0.02 0.647"/>
-<xacro:property name="vertical2_to_horizontal1_rpy" value="0 0 0"/>
-<xacro:property name="mesh_scale" value="0.001 0.001 0.001"/>
-<xacro:property name="base_visual_origin_xyz" value="0 0 0"/>
-<xacro:property name="base_collision_origin_xyz" value="0 0 0"/>
-<xacro:property name="vertical2_visual_origin_xyz" value="-0.105 -0.105 -0.722"/>
-<xacro:property name="vertical2_collision_origin_xyz" value="-0.105 -0.105 -0.722"/>
-<xacro:property name="horizontal1_visual_origin_xyz" value="0.065 -0.125 -1.369"/>
-<xacro:property name="horizontal1_collision_origin_xyz" value="0.065 -0.125 -1.369"/>
-<xacro:property name="vertical1_visual_origin_xyz" value="-0.0 -0.0 -0.012"/>
-<xacro:property name="vertical1_collision_origin_xyz" value="-0.0 -0.0 -0.012"/> -->
-<xacro:property name="base_to_vertical1_xyz" value="0.0 0.0 0.012"/>
-<xacro:property name="base_to_vertical1_rpy" value="0 0 0"/>
-<xacro:property name="vertical1_to_vertical2_xyz" value="0 0 0.71"/>
-<xacro:property name="vertical1_to_vertical2_rpy" value="0 0 0"/>
-<xacro:property name="vertical2_to_horizontal1_xyz" value="0.7 0 0"/>
-<xacro:property name="vertical2_to_horizontal1_rpy" value="0 0 0"/>
-<xacro:property name="mesh_scale" value="0.001 0.001 0.001"/>
-<xacro:property name="base_visual_origin_xyz" value="0 0 0"/>
-<xacro:property name="base_collision_origin_xyz" value="0 0 0"/>
-<xacro:property name="vertical2_visual_origin_xyz" value="0 0 -0.722"/>
-<xacro:property name="vertical2_collision_origin_xyz" value="0 0 -0.722"/>
-<xacro:property name="horizontal1_visual_origin_xyz" value="-0.7 0 -0.72"/>
-<xacro:property name="horizontal1_collision_origin_xyz" value="0 0 -0.72"/>
-<xacro:property name="vertical1_visual_origin_xyz" value="-0.0 -0.0 -0.012"/>
-<xacro:property name="vertical1_collision_origin_xyz" value="-0.0 -0.0 -0.012"/>
-<gazebo>
-  <plugin name="gazebo_ros2_control" filename="libgazebo_ros2_control.so"/>
-</gazebo>
-<link name="base_link">
-  <inertial>
-    <origin xyz="4.288906000090392e-17 2.144453000045196e-17 0.006000000000000001" rpy="0 0 0"/>
-    <mass value="6.658605629283565"/>
-    <inertia ixx="0.037535" iyy="0.037535" izz="0.074909" ixy="0.0" iyz="0.0" ixz="0.0"/>
-  </inertial>
-  <visual>
-    <origin xyz="${base_visual_origin_xyz}" rpy="0 0 0"/>
-    <geometry>
-      <mesh filename="file://$(find firebot_arm_pkg)/meshes/base_link.stl" scale="${mesh_scale}"/>
-    </geometry>
-    <material name="silver"/>
-  </visual>
-  <collision>
-    <origin xyz="${base_collision_origin_xyz}" rpy="0 0 0"/>
-    <geometry>
-      <mesh filename="file://$(find firebot_arm_pkg)/meshes/base_link.stl" scale="${mesh_scale}"/>
-    </geometry>
-  </collision>
-</link>
-<link name="linkvertical2_1">
-  <inertial>
-    <origin xyz="-0.10499999999999998 -0.10833033334588331 -0.024647039210627608" rpy="0 0 0"/>
-    <mass value="22.200698974756893"/>
-    <inertia ixx="0.120664" iyy="0.121156" izz="0.231556" ixy="-0.0" iyz="0.000483" ixz="0.0"/>
-  </inertial>
-  <visual>
-    <origin xyz="${vertical2_visual_origin_xyz}" rpy="0 0 0"/>
-    <geometry>
-      <mesh filename="file://$(find firebot_arm_pkg)/meshes/linkvertical2_1.stl" scale="${mesh_scale}"/>
-    </geometry>
-    <material name="silver"/>
-  </visual>
-  <collision>
-    <origin xyz="${vertical2_collision_origin_xyz}" rpy="0 0 0"/>
-    <geometry>
-      <mesh filename="file://$(find firebot_arm_pkg)/meshes/linkvertical2_1.stl" scale="${mesh_scale}"/>
-    </geometry>
-  </collision>
-</link>
-<link name="linkhorizontal1_1">
-  <inertial>
-    <origin xyz="0.6580876662919757 -0.12129223916653174 -0.6485017566986815" rpy="0 0 0"/>
-    <mass value="64.5078521087531"/>
-    <inertia ixx="0.463187" iyy="4.315019" izz="4.195976" ixy="0.08206" iyz="0.004506" ixz="0.022093"/>
-  </inertial>
-  <visual>
-    <origin xyz="${horizontal1_visual_origin_xyz}" rpy="0 0 0"/>
-    <geometry>
-      <mesh filename="file://$(find firebot_arm_pkg)/meshes/linkhorizontal1_1.stl" scale="${mesh_scale}"/>
-    </geometry>
-    <material name="silver"/>
-  </visual>
-  <collision>
-    <origin xyz="${horizontal1_collision_origin_xyz}" rpy="0 0 0"/>
-    <geometry>
-      <mesh filename="file://$(find firebot_arm_pkg)/meshes/linkhorizontal1_1.stl" scale="${mesh_scale}"/>
-    </geometry>
-  </collision>
-</link>
-<link name="linkvertical1_1">
-  <inertial>
-    <origin xyz="-1.4739419594933348e-17 -2.9478839189866696e-17 0.2748543377105598" rpy="0 0 0"/>
-    <mass value="19.37534476967245"/>
-    <inertia ixx="1.238356" iyy="1.238356" izz="0.290239" ixy="0.0" iyz="-0.0" ixz="0.0"/>
-  </inertial>
-  <visual>
-    <origin xyz="${vertical1_visual_origin_xyz}" rpy="0 0 0"/>
-    <geometry>
-      <mesh filename="file://$(find firebot_arm_pkg)/meshes/linkvertical1_1.stl" scale="${mesh_scale}"/>
-    </geometry>
-    <material name="silver"/>
-  </visual>
-  <collision>
-    <origin xyz="${vertical1_collision_origin_xyz}" rpy="0 0 0"/>
-    <geometry>
-      <mesh filename="file://$(find firebot_arm_pkg)/meshes/linkvertical1_1.stl" scale="${mesh_scale}"/>
-    </geometry>
-  </collision>
-</link>
-<joint name="linkvertical2_to_linkvertical1" type="prismatic">
-  <origin xyz="${vertical1_to_vertical2_xyz}" rpy="${vertical1_to_vertical2_rpy}"/>
-  <parent link="linkvertical1_1"/>
-  <child link="linkvertical2_1"/>
-  <axis xyz="0.0 0.0 1.0"/>
-  <limit upper="0.0" lower="-0.65" effort="100" velocity="100"/>
-</joint>
-<joint name="linkhorizontal1_to_linkvertical2" type="prismatic">
-  <origin xyz="${vertical2_to_horizontal1_xyz}" rpy="${vertical2_to_horizontal1_rpy}"/>
-  <parent link="linkvertical2_1"/>
-  <child link="linkhorizontal1_1"/>
-  <axis xyz="-1.0 0.0 0.0"/>
-  <limit upper="0.48" lower="0.05" effort="100" velocity="100"/>
-</joint>
-<joint name="linkvertical1_to_base_link" type="continuous">
-  <origin xyz="${base_to_vertical1_xyz}" rpy="${base_to_vertical1_rpy}"/>
-  <parent link="base_link"/>
-  <child link="linkvertical1_1"/>
-  <axis xyz="0.0 0.0 1.0"/>
-</joint>
-<ros2_control name="montagem_control" type="system">
-  <hardware>
-    <plugin>gazebo_ros2_control/GazeboSystem</plugin>
-  </hardware>
-  <joint name="linkvertical1_to_base_link">
-    <state_interface name="position"/>
-    <command_interface name="position"/>
+  <!-- Inclui arquivos Xacro externos -->
+  <xacro:include filename="$(find firebot_arm_pkg)/urdf/materials.xacro" />
+  <xacro:include filename="$(find firebot_arm_pkg)/urdf/montagem.trans" />
+  <xacro:include filename="$(find firebot_arm_pkg)/urdf/montagem.gazebo" />
+  <xacro:include filename="$(find firebot_arm_pkg)/urdf/montagem.control.xacro" />
+  <!-- Propriedades geométricas e de transformação entre links -->
+  <xacro:property name="base_to_vertical1_xyz" value="0.0 0.0 0.012"/>
+  <!-- Define a posição (xyz) da junta que conecta o link base ao primeiro link vertical, ajustando a elevação em z para compensar a base do robô. -->
+  <xacro:property name="base_to_vertical1_rpy" value="0 0 0"/>
+  <xacro:property name="vertical1_to_vertical2_xyz" value="0 0 0.71"/>
+  <!-- Define a posição (xyz) relativa entre o primeiro e o segundo link vertical, especificando o deslocamento em z necessário. -->
+  <xacro:property name="vertical1_to_vertical2_rpy" value="0 0 0"/>
+  <xacro:property name="vertical2_to_horizontal1_xyz" value="0.7 0 0"/>
+  <!-- Especifica o deslocamento em x entre o segundo link vertical e o link horizontal, indicando a extensão do braço horizontalmente. -->
+  <xacro:property name="vertical2_to_horizontal1_rpy" value="0 0 0"/>
+  <xacro:property name="mesh_scale" value="0.001 0.001 0.001"/>
+  <!-- Fator de escala aplicado às malhas STL dos links para ajustar o tamanho ao modelo desejado. -->
+  <!-- Origem visual e de colisão dos links -->
+  <xacro:property name="base_visual_origin_xyz" value="0 0 0"/>
+  <xacro:property name="base_collision_origin_xyz" value="0 0 0"/>
+  <xacro:property name="vertical2_visual_origin_xyz" value="0 0 -0.722"/>
+  <xacro:property name="vertical2_collision_origin_xyz" value="0 0 -0.722"/>
+  <xacro:property name="horizontal1_visual_origin_xyz" value="-0.7 0 -0.72"/>
+  <!-- Define a origem visual em x do link horizontal, compensando a extensão em x do braço horizontal. -->
+  <xacro:property name="horizontal1_collision_origin_xyz" value="0 0 -0.72"/>
+  <!-- Define a origem de colisão para o link horizontal, necessária para cálculos físicos. -->
+  <xacro:property name="vertical1_visual_origin_xyz" value="-0.0 -0.0 -0.012"/>
+  <xacro:property name="vertical1_collision_origin_xyz" value="-0.0 -0.0 -0.012"/>
+  <!-- Configuração de controle do Gazebo -->
+  <gazebo>
+    <plugin name="gazebo_ros2_control" filename="libgazebo_ros2_control.so"/>
+  </gazebo>
+  <!-- Definição do link base -->
+  <link name="base_link">
+    <inertial>
+      <origin xyz="4.288906000090392e-17 2.144453000045196e-17 0.006000000000000001" rpy="0 0 0"/>
+      <mass value="6.658605629283565"/>
+      <inertia ixx="0.037535" iyy="0.037535" izz="0.074909" ixy="0.0" iyz="0.0" ixz="0.0"/>
+    </inertial>
+    <visual>
+      <origin xyz="${base_visual_origin_xyz}" rpy="0 0 0"/>
+      <geometry>
+        <mesh filename="file://$(find firebot_arm_pkg)/meshes/base_link.stl" scale="${mesh_scale}"/>
+      </geometry>
+      <material name="silver"/>
+    </visual>
+    <collision>
+      <origin xyz="${base_collision_origin_xyz}" rpy="0 0 0"/>
+      <geometry>
+        <mesh filename="file://$(find firebot_arm_pkg)/meshes/base_link.stl" scale="${mesh_scale}"/>
+      </geometry>
+    </collision>
+  </link>
+  <!-- Link vertical intermediário -->
+  <link name="linkvertical2_1">
+    <inertial>
+      <origin xyz="-0.10499999999999998 -0.10833033334588331 -0.024647039210627608" rpy="0 0 0"/>
+      <mass value="22.200698974756893"/>
+      <inertia ixx="0.120664" iyy="0.121156" izz="0.231556" ixy="-0.0" iyz="0.000483" ixz="0.0"/>
+    </inertial>
+    <visual>
+      <origin xyz="${vertical2_visual_origin_xyz}" rpy="0 0 0"/>
+      <geometry>
+        <mesh filename="file://$(find firebot_arm_pkg)/meshes/linkvertical2_1.stl" scale="${mesh_scale}"/>
+      </geometry>
+      <material name="silver"/>
+    </visual>
+    <collision>
+      <origin xyz="${vertical2_collision_origin_xyz}" rpy="0 0 0"/>
+      <geometry>
+        <mesh filename="file://$(find firebot_arm_pkg)/meshes/linkvertical2_1.stl" scale="${mesh_scale}"/>
+      </geometry>
+    </collision>
+  </link>
+  <!-- Link horizontal principal -->
+  <link name="linkhorizontal1_1">
+    <inertial>
+      <origin xyz="0.6580876662919757 -0.12129223916653174 -0.6485017566986815" rpy="0 0 0"/>
+      <mass value="64.5078521087531"/>
+      <inertia ixx="0.463187" iyy="4.315019" izz="4.195976" ixy="0.08206" iyz="0.004506" ixz="0.022093"/>
+    </inertial>
+    <visual>
+      <origin xyz="${horizontal1_visual_origin_xyz}" rpy="0 0 0"/>
+      <geometry>
+        <mesh filename="file://$(find firebot_arm_pkg)/meshes/linkhorizontal1_1.stl" scale="${mesh_scale}"/>
+      </geometry>
+      <material name="silver"/>
+    </visual>
+    <collision>
+      <origin xyz="${horizontal1_collision_origin_xyz}" rpy="0 0 0"/>
+      <geometry>
+        <mesh filename="file://$(find firebot_arm_pkg)/meshes/linkhorizontal1_1.stl" scale="${mesh_scale}"/>
+      </geometry>
+    </collision>
+  </link>
+  <!-- Primeiro link vertical -->
+  <link name="linkvertical1_1">
+    <inertial>
+      <origin xyz="-1.4739419594933348e-17 -2.9478839189866696e-17 0.2748543377105598" rpy="0 0 0"/>
+      <mass value="19.37534476967245"/>
+      <inertia ixx="1.238356" iyy="1.238356" izz="0.290239" ixy="0.0" iyz="-0.0" ixz="0.0"/>
+    </inertial>
+    <visual>
+      <origin xyz="${vertical1_visual_origin_xyz}" rpy="0 0 0"/>
+      <geometry>
+        <mesh filename="file://$(find firebot_arm_pkg)/meshes/linkvertical1_1.stl" scale="${mesh_scale}"/>
+      </geometry>
+      <material name="silver"/>
+    </visual>
+    <collision>
+      <origin xyz="${vertical1_collision_origin_xyz}" rpy="0 0 0"/>
+      <geometry>
+        <mesh filename="file://$(find firebot_arm_pkg)/meshes/linkvertical1_1.stl" scale="${mesh_scale}"/>
+      </geometry>
+    </collision>
+  </link>
+  <!-- Juntas conectando os links -->
+  <joint name="linkvertical2_to_linkvertical1" type="prismatic">
+    <origin xyz="${vertical1_to_vertical2_xyz}" rpy="${vertical1_to_vertical2_rpy}"/>
+    <parent link="linkvertical1_1"/>
+    <child link="linkvertical2_1"/>
+    <axis xyz="0.0 0.0 1.0"/>
+    <limit upper="0.0" lower="-0.65" effort="100" velocity="100"/>
   </joint>
-  <joint name="linkvertical2_to_linkvertical1">
-    <state_interface name="position"/>
-    <command_interface name="position"/>
+  <joint name="linkhorizontal1_to_linkvertical2" type="prismatic">
+    <origin xyz="${vertical2_to_horizontal1_xyz}" rpy="${vertical2_to_horizontal1_rpy}"/>
+    <parent link="linkvertical2_1"/>
+    <child link="linkhorizontal1_1"/>
+    <axis xyz="-1.0 0.0 0.0"/>
+    <limit upper="0.48" lower="0.05" effort="100" velocity="100"/>
   </joint>
-  <joint name="linkhorizontal1_to_linkvertical2">
-    <state_interface name="position"/>
-    <command_interface name="position"/>
+  <joint name="linkvertical1_to_base_link" type="continuous">
+    <origin xyz="${base_to_vertical1_xyz}" rpy="${base_to_vertical1_rpy}"/>
+    <parent link="base_link"/>
+    <child link="linkvertical1_1"/>
+    <axis xyz="0.0 0.0 1.0"/>
   </joint>
-</ros2_control>
-<link name="dummy_base_inertia">
+  <!-- Configuração de controle para os joints -->
+  <ros2_control name="montagem_control" type="system">
+    <hardware>
+      <plugin>gazebo_ros2_control/GazeboSystem</plugin>
+    </hardware>
+    <joint name="linkvertical1_to_base_link">
+      <state_interface name="position"/>
+      <command_interface name="position"/>
+    </joint>
+    <joint name="linkvertical2_to_linkvertical1">
+      <state_interface name="position"/>
+      <command_interface name="position"/>
+    </joint>
+    <joint name="linkhorizontal1_to_linkvertical2">
+      <state_interface name="position"/>
+      <command_interface name="position"/>
+    </joint>
+  </ros2_control>
+  <!-- Links e juntas dummy para compensar inércia e centralizar o modelo -->
+  <link name="dummy_base_inertia">
   <inertial>
     <mass value="0.1"/>

Commit message: Ajustes controle

File: install/firebot_arm_pkg/share/firebot_arm_pkg/urdf/montagem.control.xacro (robot description, xacro)
@@ -1,31 +1,23 @@
 <?xml version="1.0" ?>
 <robot xmlns:xacro="http://www.ros.org/wiki/xacro">
-  <!-- Configurações ros2_control para 3 juntas -->
-  <ros2_control name="montagem_control" type="system">
-    <!-- Definição do plugin que conecta o controle ros2_control ao simulador Gazebo -->
+<ros2_control name="GazeboSystem" type="system">
     <hardware>
-      <plugin>gazebo_ros2_control/GazeboSystem</plugin>
+        <plugin>gazebo_ros2_control/GazeboSystem</plugin>
     </hardware>
-    <!-- Definição da primeira junta: linkvertical1_to_base_link -->
     <joint name="linkvertical1_to_base_link">
-      <!-- Interface de estado usada para monitorar a posição da junta -->
-      <state_interface name="position"/>
-      <!-- Interface de comando usada para controlar a posição da junta -->
-      <command_interface name="position"/>
+        <command_interface name="position"/>
+        <state_interface name="position"/>
+        <state_interface name="velocity"/>
     </joint>
-    <!-- Definição da segunda junta: linkvertical2_to_linkvertical1 -->
     <joint name="linkvertical2_to_linkvertical1">
-      <!-- Interface de estado usada para monitorar a posição da junta -->
-      <state_interface name="position"/>
-      <!-- Interface de comando usada para controlar a posição da junta -->
-      <command_interface name="position"/>
+        <command_interface name="position"/>
+        <state_interface name="position"/>
+        <state_interface name="velocity"/>
     </joint>
-    <!-- Definição da terceira junta: linkhorizontal1_to_linkvertical2 -->
     <joint name="linkhorizontal1_to_linkvertical2">
-      <!-- Interface de estado usada para monitorar a posição da junta -->
-      <state_interface name="position"/>
-      <!-- Interface de comando usada para controlar a posição da junta -->
-      <command_interface name="position"/>
+        <command_interface name="position"/>
+        <state_interface name="position"/>
+        <state_interface name="velocity"/>
     </joint>
-  </ros2_control>
+</ros2_control>
 </robot>

File: install/firebot_arm_pkg/share/firebot_arm_pkg/urdf/montagem.xacro (robot description, xacro)
@@ -138,22 +138,4 @@
     <axis xyz="0.0 0.0 1.0"/>
   </joint>
-  <!-- Configuração de controle para os joints -->
-  <ros2_control name="montagem_control" type="system">
-    <hardware>
-      <plugin>gazebo_ros2_control/GazeboSystem</plugin>
-    </hardware>
-    <joint name="linkvertical1_to_base_link">
-      <state_interface name="position"/>
-      <command_interface name="position"/>
-    </joint>
-    <joint name="linkvertical2_to_linkvertical1">
-      <state_interface name="position"/>
-      <command_interface name="position"/>
-    </joint>
-    <joint name="linkhorizontal1_to_linkvertical2">
-      <state_interface name="position"/>
-      <command_interface name="position"/>
-    </joint>
-  </ros2_control>
   <!-- Links e juntas dummy para compensar inércia e centralizar o modelo -->
   <link name="dummy_base_inertia">
